File: ipod/ipod.kicad_sch (KiCad schematic)
At the start: 0 parts

Commit message: feat: add fan header footprint and update PCB project configuration files
Parts:
- added J1: Conn_01x04_Pin, Connector:FanPinHeader_1x04_P2.54mm_Vertical, symbol Connector:Conn_01x04_Pin
- added U1: ESP32-S3-WROOM-1, RF_Module:ESP32-S3-WROOM-1, symbol RF_Module:ESP32-S3-WROOM-1
- added U2: CR2013-MI2120, Display:CR2013-MI2120, symbol Driver_Display:CR2013-MI2120
- added U3: PCM5102A, Package_SO:TSSOP-20_4.4x6.5mm_P0.65mm, symbol Audio:PCM5102A
Connections:
- new net: U1.12 (IO8), U2.4 (RESET)
- new net: U1.17 (IO9), U2.5 (D/~{C})
- new net: U1.18 (IO10), U2.3 (~{CS})
- new net: U1.19 (IO11), U2.6 (MOSI)
- new net: U1.20 (IO12), U2.7 (SCK)
- new net: U1.21 (IO13), U2.9 (MISO)
- new net: U1.22 (IO14), U3.13 (BCK)
- new net: J1.4 (Pin_4), U1.38 (IO2)
- new net: J1.3 (Pin_3), U1.39 (IO1)
- new net: U1.8 (IO15), U3.15 (LRCK)
- new net: U1.9 (IO16), U3.14 (DIN)
- new net +3V3: J1.1 (Pin_1), U1.2 (3V3), U2.1 (VCC), U2.8 (LED), U3.17 (XSMT)
- new net GND: J1.2 (Pin_2), U1.1 (GND), U1.40 (GND), U1.41 (GND), U2.2 (GND), U3.12 (SCK), U3.16 (FMT)
- no-connect marks 0 -> 45
